Commit message: build URDF joints

File: urdf/my_robot.urdf (robot description, URDF)
Before this commit: robot my_robot, 1 links, 0 joints
Links:
- added link shoulder_link; visual cylinder length=0.3 radius=0.1
Joints:
- added joint base_shoulder_joint: type fixed, parent base_link, child shoulder_link, origin xyz=0 0.5 0.3 rpy=0 0 0

Commit message: describe joint origin location

File: urdf/my_robot.urdf (robot description, URDF)
Before this commit: robot my_robot, 2 links, 1 joints
Joints:
- joint base_shoulder_joint: origin xyz=0 0.5 0.3 rpy=0 0 0 -> xyz=0 0 0.2 rpy=0 0 0
