Commit message: finish my_robot urdf

File: urdf/my_robot_preliminary.urdf (robot description, URDF)
Before this commit: robot my_robot, 2 links, 1 joints
Joints:
- joint base_shoulder_joint: axis 0 0 1 -> (none); limit lower=-3.14 upper=3.14 effort=100 velocity=100 -> (none); type revolute -> fixed
