Commit message: rename left right

File: urdf/robot_car.urdf (robot description, URDF)
Before this commit: robot robot_car, 2 links, 1 joints
Joints:
- joint base_left_wheel_joint: child right_wheel -> left_wheel

Commit message: car theoretically finished

File: urdf/robot_car.urdf (robot description, URDF)
Before this commit: robot robot_car, 2 links, 1 joints
Links:
- removed link left_wheel
- added link left_wheel_link; visual cylinder length=0.05 radius=0.2
- added link right_wheel_link; visual cylinder length=0.05 radius=0.2
- added link support_wheel_link; visual sphere radius=0.05
Joints:
- added joint base_right_wheel_joint: type continuous, parent base_link, child right_wheel_link, origin xyz=-0.1 -0.225 0.2 rpy=0 0 0, axis 0 1 0
- added joint base_support_wheel_joint: type fixed, parent base_link, child support_wheel_link, origin xyz=0.2 0 0.05 rpy=0 0 0
- joint base_left_wheel_joint: axis 0 0 1 -> 0 1 0; child left_wheel -> left_wheel_link; origin xyz=-0.1 0.225 0.2 rpy=-1.57 0 0 -> xyz=-0.1 0.225 0.2 rpy=0 0 0
